Commit message: IMU and GPS added, StereoCamera and final editing pending

File: src/roverbot/urdf/roverbot.xacro (robot description, xacro)
@@ -133,5 +133,5 @@
 		</collision>
 	</link>
-	<!-- Camera -->
+	<!-- CAMERA LINK -->
 	<link name="camera">
 		<inertial>
@@ -157,5 +157,5 @@
 		</collision>
 	</link>
-	<!-- Hokuyo Lidar -->
+	<!-- LIDAR LINK -->
 	<link name="hokuyo">
 		<inertial>
@@ -181,4 +181,45 @@
 		</collision>
 	</link>
+	<!-- IMU LINK -->
+	<link name="imu_link">
+    <visual>
+      <geometry>
+        <box size="0.15 0.15 0.05"/>
+      </geometry>
+    </visual>
+    <collision>
+      <geometry>
+        <box size="0.15 0.15 0.05"/>
+      </geometry>
+    </collision>
+    <inertial>
+      <mass value="1e-5" />
+      <origin xyz="0 0 0" rpy="0 0 0"/>
+      <inertia ixx="1e-6" ixy="0" ixz="0" iyy="1e-6" iyz="0" izz="1e-6" />
+    </inertial>
+  </link>
+   	<!-- GPS LINK -->
+   	  <link name="gps_link">
+    <collision>
+      <origin xyz="0 0 0.1" rpy="0 0 0"/>
+      <geometry>
+        <box size="0.1 0.1 0.1"/>
+      </geometry>
+    </collision>
+    <visual>
+      <origin xyz="-0.1 0 0.1" rpy="0 0 0"/>
+      <geometry>
+        <cylinder radius="0.05" length="0.05"/>
+      </geometry>
+    </visual>
+    <inertial>
+      <origin xyz="0 0 0.1" rpy="0 0 0"/>
+      <mass value="1"/>
+      <inertia
+        ixx="1.0" ixy="0.0" ixz="0.0"
+        iyy="1.0" iyz="0.0"
+        izz="1.0"/>
+    </inertial>
+  </link>
 	<!-- Project center to the ground -->
 	<link name="robot_footprint"></link>
@@ -220,5 +261,5 @@
 	    <dynamics damping="1.0" friction="1.0" />
 	</joint>
-	<!-- Camera Joint -->
+	<!-- CAMERA JOINT -->
 	<joint name="camera_joint" type="fixed">
 		<origin xyz="0.26 0 0" rpy="0 0 0" />
@@ -227,5 +268,5 @@
 		<axis xyz="0 1 0"/>
 	</joint>
-	<!-- Hokoyu Joint -->
+	<!-- LIDAR JOINT -->
 	<joint name="hokuyo_joint" type="fixed">
 	    <origin xyz="0.2 0 0.2" rpy="0 0 0" />
@@ -234,4 +275,18 @@
 	    <axis xyz="0 1 0"/>
 	</joint>
+	<!-- IMU JOINT -->
+	<joint name="imu_joint" type="fixed">
+    <origin xyz="0.04 0 0.12" rpy="0 0 0" />
+    <parent link="chassis"/>
+    <child link="imu_link" />
+    <axis xyz="0 1 0"/>
+  </joint>
+  	<!--GPS JOINT -->
+  	 <joint name="gps_joint" type="fixed">
+    <origin xyz="0.4 0.0 0.04" rpy="0 0 0" />
+    <parent link="robot_footprint"/>
+    <child link="gps_link" />
+    <axis xyz="0 1 0"/>
+  </joint>
 	<joint name="robot_footprint_joint" type="fixed">
 		<origin xyz="0 0 0" rpy="0 0 0" />
@@ -282,4 +337,7 @@
 		<material>Gazebo/Red</material>
 	</gazebo>
+	<gazebo reference="imu_link">
+		<material>Gazebo/Orange</material>
+	</gazebo>
 	<gazebo reference="chassis">
 		<material>Gazebo/Blue</material>

Commit message: ZED 2 Stereocamera Plugin Added

File: src/roverbot/urdf/roverbot.xacro (robot description, xacro)
@@ -222,4 +222,22 @@
     </inertial>
   </link>
+  	<!-- ZED 2 LINK -->
+  	 <link name="ZED2">
+    <visual>
+      <geometry>
+        <box size="0.05 0.1 0.05"/>
+      </geometry>
+    </visual>
+    <collision>
+      <geometry>
+        <box size="0.05 0.1 0.05"/>
+      </geometry>
+    </collision>
+    <inertial>
+      <mass value="1e-5" />
+      <origin xyz="0 0 0" rpy="0 0 0"/>
+      <inertia ixx="1e-6" ixy="0" ixz="0" iyy="1e-6" iyz="0" izz="1e-6" />
+    </inertial>
+  </link>
 	<!-- Project center to the ground -->
 	<link name="robot_footprint"></link>
@@ -254,17 +272,17 @@
 	<!-- Left Wheel Joint Front-->
 	<joint type="continuous" name="left_wheel_hinge_front">
-	    <origin xyz="0.2 0.30 0" rpy="0 0 0" />
-	    <parent link="chassis"/>
-	    <child link="left_wheel_front" />
-	    <axis xyz="0 1 0" rpy="0 0 0" />
-	    <limit effort="10000" velocity="1000" />
-	    <dynamics damping="1.0" friction="1.0" />
+	<origin xyz="0.2 0.30 0" rpy="0 0 0" />
+	<parent link="chassis"/>
+	<child link="left_wheel_front" />
+	<axis xyz="0 1 0" rpy="0 0 0" />
+	<limit effort="10000" velocity="1000" />
+	<dynamics damping="1.0" friction="1.0" />
 	</joint>
 	<!-- CAMERA JOINT -->
 	<joint name="camera_joint" type="fixed">
-		<origin xyz="0.26 0 0" rpy="0 0 0" />
-		<parent link="chassis"/>
-		<child link="camera" />
-		<axis xyz="0 1 0"/>
+	<origin xyz="0.26 0 0" rpy="0 0 0" />
+	<parent link="chassis"/>
+	<child link="camera" />
+	<axis xyz="0 1 0"/>
 	</joint>
 	<!-- LIDAR JOINT -->
@@ -277,16 +295,23 @@
 	<!-- IMU JOINT -->
 	<joint name="imu_joint" type="fixed">
-    <origin xyz="0.04 0 0.12" rpy="0 0 0" />
-    <parent link="chassis"/>
-    <child link="imu_link" />
-    <axis xyz="0 1 0"/>
-  </joint>
+    	<origin xyz="0.04 0 0.12" rpy="0 0 0" />
+    	<parent link="chassis"/>
+    	<child link="imu_link" />
+    	<axis xyz="0 1 0"/>
+  	</joint>
   	<!--GPS JOINT -->
-  	 <joint name="gps_joint" type="fixed">
-    <origin xyz="0.4 0.0 0.04" rpy="0 0 0" />
-    <parent link="robot_footprint"/>
-    <child link="gps_link" />
-    <axis xyz="0 1 0"/>
-  </joint>
+  	<joint name="gps_joint" type="fixed">
+    	<origin xyz="0.4 0.0 0.04" rpy="0 0 0" />
+    	<parent link="robot_footprint"/>
+    	<child link="gps_link" />
+   	 <axis xyz="0 1 0"/>
+  	</joint>
+  	<!-- ZED2 JOINT -->
+  	<joint name="ZED2_joint" type="fixed">
+  	<origin xyz ="-0.15 0 0.195" rpy ="0 0 0" />
+  	<parent link="robot_footprint"/>
+  	<child link ="ZED2" />
+  	<axis xyz ="0 1 0" />
+  	</joint>
 	<joint name="robot_footprint_joint" type="fixed">
 		<origin xyz="0 0 0" rpy="0 0 0" />
@@ -331,11 +356,8 @@
 		<minDepth>0.00</minDepth>
 	</gazebo>
-	<!--<gazebo reference="right_wheel">
-		<material>Gazebo/Green</material>
-	</gazebo>-->
 	<gazebo reference="camera">
 		<material>Gazebo/Red</material>
 	</gazebo>
-	<gazebo reference="imu_link">
+	<gazebo reference="ZED2">
 		<material>Gazebo/Orange</material>
 	</gazebo>
@@ -343,5 +365,5 @@
 		<material>Gazebo/Blue</material>
 	</gazebo>
-	<!-- Motor, Camera and Lidar Simulation -->
+	<!-- Sensors, Camera and Lidar Simulation -->
 	<xacro:include filename="$(find roverbot)/urdf/roverbot.gazebo" />
 </robot>
